Commit message: 切换新的模型与配置文件

File: src/z_arm_2442c0_model/src/config/z_arm_2442c0.ros2_control.xacro (robot description, xacro)
@@ -8,40 +8,33 @@
                 <plugin>mock_components/GenericSystem</plugin>
             </hardware>
-            <joint name="fixed_lift_joint">
+            <joint name="lift_joint">
                 <command_interface name="position"/>
                 <state_interface name="position">
-                  <param name="initial_value">${initial_positions['fixed_lift_joint']}</param>
+                  <param name="initial_value">${initial_positions['lift_joint']}</param>
                 </state_interface>
                 <state_interface name="velocity"/>
             </joint>
-            <joint name="lift_revo_joint">
+            <joint name="revolute_1_joint">
                 <command_interface name="position"/>
                 <state_interface name="position">
-                  <param name="initial_value">${initial_positions['lift_revo_joint']}</param>
+                  <param name="initial_value">${initial_positions['revolute_1_joint']}</param>
                 </state_interface>
                 <state_interface name="velocity"/>
             </joint>
-            <joint name="double_revo_1_joint">
+            <joint name="revolute_2_jointt">
                 <command_interface name="position"/>
                 <state_interface name="position">
-                  <param name="initial_value">${initial_positions['double_revo_1_joint']}</param>
+                  <param name="initial_value">${initial_positions['revolute_2_joint']}</param>
                 </state_interface>
                 <state_interface name="velocity"/>
             </joint>
-            <joint name="double_revo_2_joint">
+            <joint name="revolute_3_joint">
                 <command_interface name="position"/>
                 <state_interface name="position">
-                  <param name="initial_value">${initial_positions['double_revo_2_joint']}</param>
+                  <param name="initial_value">${initial_positions['revolute_3_joint']}</param>
                 </state_interface>
                 <state_interface name="velocity"/>
             </joint>
-            <joint name="camera_1_joint">
-                <command_interface name="position"/>
-                <state_interface name="position">
-                  <param name="initial_value">0.0</param>
-                </state_interface>
-                <state_interface name="velocity"/>
-            </joint>
-            <joint name="camera_2_joint">
+            <joint name="camera_1_rot_joint">
                 <command_interface name="position"/>
                 <state_interface name="position">

File: src/z_arm_2442c0_model/src/urdf/z_arm_2442c0.urdf (robot description, URDF)
Before this commit: robot z_arm_2442c0, 10 links, 9 joints
Links:
- removed link fixed_link
- added link base_lift_link, mass 2.24198664042392; collision mesh filename=package://z_arm_2442c0_model/meshes/base_lift_link.STL; visual mesh filename=package://z_arm_2442c0_model/meshes/base_lift_link.STL
- added link camera_1_rot_link; visual box size=0.001 0.001 0.001
- added link camera_3_link, mass 1.45710864588612; collision mesh filename=package://z_arm_2442c0_model/meshes/camera_3_link.STL; visual mesh filename=package://z_arm_2442c0_model/meshes/camera_3_link.STL
- link base_link: mass 1311.6 -> 951.87; geometry collision mesh filename=package://z_arm_2442c0_model/meshes/base_link.STL; visual mesh filename=package://z_arm_2442c0_model/meshes/base_link.STL
- link camera_1_link: mass 1.4455 -> 0.0230681246047575; geometry collision mesh filename=package://z_arm_2442c0_model/meshes/camera_1_link.STL; visual mesh filename=package://z_arm_2442c0_model/meshes/camera_1_link.STL
- link camera_2_link: mass 0.023068 -> 0.0230681244154274; geometry collision mesh filename=package://z_arm_2442c0_model/meshes/camera_2_link.STL; visual mesh filename=package://z_arm_2442c0_model/meshes/camera_2_link.STL
- link camera_base_link: mass 2.6147 -> 0.321807581331945; geometry collision mesh filename=package://z_arm_2442c0_model/meshes/camera_base_link.STL; visual mesh filename=package://z_arm_2442c0_model/meshes/camera_base_link.STL
- link door_link: mass 85.7009910260309 -> 181.651646287815; geometry collision mesh filename=package://z_arm_2442c0_model/meshes/door_link.STL; visual mesh filename=package://z_arm_2442c0_model/meshes/door_link.STL
- link lift_link: mass 0.99372 -> 0.993724555380008; geometry collision mesh filename=package://z_arm_2442c0_model/meshes/lift_link.STL; visual mesh filename=package://z_arm_2442c0_model/meshes/lift_link.STL
- link revolute_1_link: mass 2.3889553320756 -> 2.3889549988802; geometry collision mesh filename=package://z_arm_2442c0_model/meshes/revolute_1_link.STL; visual mesh filename=package://z_arm_2442c0_model/meshes/revolute_1_link.STL
- link revolute_2_link: mass 1.22952478849448 -> 1.2295144495631; geometry collision mesh filename=package://z_arm_2442c0_model/meshes/revolute_2_link.STL; visual mesh filename=package://z_arm_2442c0_model/meshes/revolute_2_link.STL
- link revolute_3_link: mass 0.0445549065270102 -> 0.0445549065520843; geometry collision mesh filename=package://z_arm_2442c0_model/meshes/revolute_3_link.STL; visual mesh filename=package://z_arm_2442c0_model/meshes/revolute_3_link.STL
Joints:
- removed joint double_revo_1_joint
- removed joint double_revo_2_joint
- removed joint fixed_joint
- removed joint fixed_lift_joint
- removed joint lift_revo_joint
- added joint base_joint: type fixed, parent base_link, child base_lift_link, origin xyz=-0.97852 0.59917 0.42459 rpy=0 0 0, axis 0 0 0
- added joint camera_1_rot_joint: type continuous, parent camera_base_link, child camera_1_rot_link, origin xyz=0.14534 0 0.13089 rpy=0 0 0, axis 0 0 1
- added joint camera_3_joint: type fixed, parent camera_1_rot_link, child camera_3_link, origin xyz=-0.00181 -0.025558 0.029 rpy=0 0 0, axis 0 0 0
- added joint lift_joint: type prismatic, parent base_lift_link, child lift_link, origin xyz=0.1207 0.0018675 0.5009 rpy=0 0 0, axis 0 0 -1, limit lower=-0.068 upper=0.268 effort=10.0 velocity=2.5
- added joint revolute_1_joint: type revolute, parent lift_link, child revolute_1_link, origin xyz=0.012024 0.00017897 -0.066 rpy=0 0 0, axis 0 0 1, limit lower=-0.550 upper=2.59 effort=10.0 velocity=2.5
- added joint revolute_2_joint: type revolute, parent revolute_1_link, child revolute_2_link, origin xyz=0.11991 -0.18445 -0.118 rpy=0 0 0, axis 0 0 -1, limit lower=-1.056 upper=4.678 effort=10.0 velocity=2.5
- added joint revolute_3_joint: type continuous, parent revolute_2_link, child revolute_3_link, origin xyz=0.1017 0.17221 -0.006 rpy=0 0 0, axis 0 0 -1
- joint camera_1_joint: axis 0 0 1 -> 0 0 0; limit lower=0.0 upper=0.001 effort=1.0 velocity=0.1 -> (none); origin xyz=-0.00041282 -0.015045 -0.2777 rpy=0 0 0 -> xyz=0.0234 0.047416 -0.0145 rpy=0 0 0; parent camera_base_link -> camera_1_rot_link; type prismatic -> fixed
- joint camera_2_joint: axis 0 0 1 -> 0 0 0; limit lower=0.0 upper=0.001 effort=1.0 velocity=0.1 -> (none); origin xyz=-0.0009298 0.056015 -0.22685 rpy=0 0 0 -> xyz=-0.0216 0.047416 -0.0145 rpy=0 0 0; parent camera_base_link -> camera_1_rot_link; type prismatic -> fixed
- joint camera_base_joint: axis (none) -> 0 0 0; origin xyz=0 0 0 rpy=0 0 0 -> xyz=0 0 -0.015655 rpy=0 0 0
- joint door_joint: axis 0 0 -1 -> 0 -1 0; limit lower=0 upper=0 effort=0 velocity=0 -> lower=-1 upper=0.268 effort=10.0 velocity=2.5; origin xyz=1.1569 -1.0402 1.341 rpy=0 0 -0.34907 -> xyz=-1.2401 0.6 1.0971 rpy=0 0 0

File: src/z_arm_2442c0_model/src/urdf/z_arm_2442c0.urdf.xacro (robot description, xacro)
@@ -13,35 +13,35 @@
     <inertial>
       <origin
-        xyz="-0.18371 -0.036956 1.0828"
-        rpy="0 0 0" />
-      <mass
-        value="1311.6" />
-      <inertia
-        ixx="604.63"
-        ixy="-8.8817"
-        ixz="27.771"
-        iyy="546.1"
-        iyz="4.8371"
-        izz="549.71" />
-    </inertial>
-    <visual>
-      <origin
-        xyz="0 0 0.044"
-        rpy="0 0 0" />
-      <geometry>
-         <mesh filename="file:///home/sunshine/project/z_arm_2442c0/install/z_arm_2442c0_model/share/z_arm_2442c0_model/meshes/base_link.STL"/>
-      </geometry>
-      <material
-        name="">
-        <color
-          rgba="1 1 1 1" />
-      </material>
-    </visual>
-    <collision>
-      <origin
-        xyz="0 0 0.044"
-        rpy="0 0 0" />
-      <geometry>
-         <mesh filename="file:///home/sunshine/project/z_arm_2442c0/install/z_arm_2442c0_model/share/z_arm_2442c0_model/meshes/base_link.STL"/>
+        xyz="-0.6178 0.59958 0.70792"
+        rpy="0 0 0" />
+      <mass
+        value="951.87" />
+      <inertia
+        ixx="137.78"
+        ixy="0.0044402"
+        ixz="-10.933"
+        iyy="119.15"
+        iyz="-0.00067217"
+        izz="158.71" />
+    </inertial>
+    <visual>
+      <origin
+        xyz="0 0 0"
+        rpy="0 0 0" />
+      <geometry>
+        <mesh filename="file://$(find z_arm_2442c0_model)/meshes/base_link.STL" />
+      </geometry>
+      <material
+        name="">
+        <color
+          rgba="1 1 1 1" />
+      </material>
+    </visual>
+    <collision>
+      <origin
+        xyz="0 0 0"
+        rpy="0 0 0" />
+      <geometry>
+        <mesh filename="file://$(find z_arm_2442c0_model)/meshes/base_link.STL" />
       </geometry>
     </collision>
@@ -51,35 +51,35 @@
     <inertial>
       <origin
-        xyz="0.000906627818809458 -0.00848429199587175 -0.0177814412093629"
-        rpy="0 0 0" />
-      <mass
-        value="85.7009910260309" />
-      <inertia
-        ixx="11.4196065030808"
-        ixy="-0.00532670528961088"
-        ixz="0.000390873878802149"
-        iyy="24.6809750482461"
-        iyz="-0.00570672117476616"
-        izz="13.5149037455903" />
-    </inertial>
-    <visual>
-      <origin
-        xyz="0.0 0.0 0.0"
-        rpy="0 0 0" />
-      <geometry>
-         <mesh filename="file:///home/sunshine/project/z_arm_2442c0/install/z_arm_2442c0_model/share/z_arm_2442c0_model/meshes/door_link.STL"/>
-      </geometry>
-      <material
-        name="">
-        <color
-          rgba="1 1 1 1" />
-      </material>
-    </visual>
-    <collision>
-      <origin
-        xyz="0.0 0.0 0.0"
-        rpy="0 0 0" />
-      <geometry>
-          <mesh filename="file:///home/sunshine/project/z_arm_2442c0/install/z_arm_2442c0_model/share/z_arm_2442c0_model/meshes/door_link.STL"/>
+        xyz="0.32048066892287 2.3834458054398E-10 0.562398088143635"
+        rpy="0 0 0" />
+      <mass
+        value="181.651646287815" />
+      <inertia
+        ixx="48.7702456064344"
+        ixy="-1.59733671105852E-10"
+        ixz="-10.9325544807547"
+        iyy="25.5516862461827"
+        iyz="1.39131607597233E-11"
+        izz="36.1437519623492" />
+    </inertial>
+    <visual>
+      <origin
+        xyz="0 0 0"
+        rpy="0 0 0" />
+      <geometry>
+        <mesh filename="file://$(find z_arm_2442c0_model)/meshes/door_link.STL" />
+      </geometry>
+      <material
+        name="">
+        <color
+          rgba="1 1 1 1" />
+      </material>
+    </visual>
+    <collision>
+      <origin
+        xyz="0 0 0"
+        rpy="0 0 0" />
+      <geometry>
+        <mesh filename="file://$(find z_arm_2442c0_model)/meshes/door_link.STL" />
       </geometry>
     </collision>
@@ -89,6 +89,6 @@
     type="revolute">
     <origin
-      xyz="1.1569 -1.0402 1.341"
-      rpy="0 0 -0.34907" />
+      xyz="-1.2401 0.6 1.0971"
+      rpy="0 0 0" />
     <parent
       link="base_link" />
@@ -96,62 +96,57 @@
       link="door_link" />
     <axis
-      xyz="0 0 -1" />
-    <limit
-      lower="0"
-      upper="0"
-      effort="0"
-      velocity="0" />
-    <dynamics damping="0.5" friction="0.1"/>
-  </joint>
-  <link
-    name="fixed_link">
-    <inertial>
-      <origin
-        xyz="-0.013691 -0.00061437 0.2572"
-        rpy="0 0 0" />
-      <mass
-        value="2.2298" />
-      <inertia
-        ixx="0.050665"
-        ixy="5.3209E-05"
-        ixz="-0.00015617"
-        iyy="0.049468"
-        iyz="-0.00057632"
-        izz="0.01024" />
-    </inertial>
-    <visual>
-      <origin
-        xyz="0 0 0"
-        rpy="0 0 0" />
-      <geometry>
-        <mesh filename="file:///home/sunshine/project/z_arm_2442c0/install/z_arm_2442c0_model/share/z_arm_2442c0_model/meshes/fixed_link.STL"/>
-      </geometry>
-      <material
-        name="">
-        <color
-          rgba="1 1 1 1" />
-      </material>
-    </visual>
-    <collision>
-      <origin
-        xyz="0 0 0"
-        rpy="0 0 0" />
-      <geometry>
-        <mesh filename="file:///home/sunshine/project/z_arm_2442c0/install/z_arm_2442c0_model/share/z_arm_2442c0_model/meshes/fixed_link.STL"/>
-      </geometry>
-    </collision>
-  </link>
-  <joint
-    name="fixed_joint"
+      xyz="0 -1 0" />
+  <limit lower="-1" upper="0.268" effort="10.0" velocity="2.5" />
+  </joint>
+  <link
+    name="base_lift_link">
+    <inertial>
+      <origin
+        xyz="-0.0138235267428053 -0.000617643429039805 0.256337391094087"
+        rpy="0 0 0" />
+      <mass
+        value="2.24198664042392" />
+      <inertia
+        ixx="0.0506641832977411"
+        ixy="7.09367963595699E-05"
+        ixz="-0.000147564343759707"
+        iyy="0.0494711018646685"
+        iyz="-0.000578573299400282"
+        izz="0.0102402545016511" />
+    </inertial>
+    <visual>
+      <origin
+        xyz="0 0 0"
+        rpy="0 0 0" />
+      <geometry>
+        <mesh filename="file://$(find z_arm_2442c0_model)/meshes/base_lift_link.STL" />
+      </geometry>
+      <material
+        name="">
+        <color
+          rgba="1 1 1 1" />
+      </material>
+    </visual>
+    <collision>
+      <origin
+        xyz="0 0 0"
+        rpy="0 0 0" />
+      <geometry>
+        <mesh filename="file://$(find z_arm_2442c0_model)/meshes/base_lift_link.STL" />
+      </geometry>
+    </collision>
+  </link>
+  <joint
+    name="base_joint"
     type="fixed">
     <origin
-      xyz="-0.225 -0.15 1.025"
+      xyz="-0.97852 0.59917 0.42459"
       rpy="0 0 0" />
     <parent
       link="base_link" />
     <child
-      link="fixed_link" />
-    <axis
-      xyz="0 0 -1" />
+      link="base_lift_link" />
+    <axis
+      xyz="0 0 0" />
   </joint>
   <link
@@ -159,52 +154,51 @@
     <inertial>
       <origin
-        xyz="0.081223 -7.7483E-05 -0.025227"
-        rpy="0 0 0" />
-      <mass
-        value="0.99372" />
-      <inertia
-        ixx="0.00095014"
-        ixy="-1.4453E-05"
-        ixz="7.3306E-05"
-        iyy="0.0034291"
-        iyz="-2.0913E-06"
-        izz="0.0039252" />
-    </inertial>
-    <visual>
-      <origin
-        xyz="0 0 0"
-        rpy="0 0 0" />
-      <geometry>
-        <mesh filename="file:///home/sunshine/project/z_arm_2442c0/install/z_arm_2442c0_model/share/z_arm_2442c0_model/meshes/lift_link.STL"/>
-      </geometry>
-      <material
-        name="">
-        <color
-          rgba="1 1 1 1" />
-      </material>
-    </visual>
-    <collision>
-      <origin
-        xyz="0 0 0"
-        rpy="0 0 0" />
-      <geometry>
-        <mesh filename="file:///home/sunshine/project/z_arm_2442c0/install/z_arm_2442c0_model/share/z_arm_2442c0_model/meshes/lift_link.STL"/>
-      </geometry>
-    </collision>
-  </link>
-  <joint
-    name="fixed_lift_joint"
+        xyz="-0.0394813607628044 -0.000736121252994326 -0.0372265212000362"
+        rpy="0 0 0" />
+      <mass
+        value="0.993724555380008" />
+      <inertia
+        ixx="0.000951122396615806"
+        ixy="-5.13373343735685E-05"
+        ixz="7.33288284051898E-05"
+        iyy="0.00342810823599992"
+        iyz="-1.00008205904848E-06"
+        izz="0.00392520888178525" />
+    </inertial>
+    <visual>
+      <origin
+        xyz="0 0 0"
+        rpy="0 0 0" />
+      <geometry>
+        <mesh filename="file://$(find z_arm_2442c0_model)/meshes/lift_link.STL" />
+      </geometry>
+      <material
+        name="">
+        <color
+          rgba="1 1 1 1" />
+      </material>
+    </visual>
+    <collision>
+      <origin
+        xyz="0 0 0"
+        rpy="0 0 0" />
+      <geometry>
+        <mesh filename="file://$(find z_arm_2442c0_model)/meshes/lift_link.STL" />
+      </geometry>
+    </collision>
+  </link>
+  <joint
+    name="lift_joint"
     type="prismatic">
     <origin
-      xyz="0 0 0.4889"
+      xyz="0.1207 0.0018675 0.5009"
       rpy="0 0 0" />
     <parent
-      link="fixed_link" />
+      link="base_lift_link" />
     <child
       link="lift_link" />
     <axis
       xyz="0 0 -1" />
-  <limit lower="-0.068" upper="0.268" effort="10.0" velocity="2.5" />
-  <dynamics damping="0.5" friction="0.1"/>
+    <limit lower="-0.068" upper="0.268" effort="10.0" velocity="2.5" />
   </joint>
   <link
@@ -212,44 +206,44 @@
     <inertial>
       <origin
-        xyz="0.0759324011920596 -0.0813064180574647 0.0368742891101176"
-        rpy="0 0 0" />
-      <mass
-        value="2.3889553320756" />
-      <inertia
-        ixx="0.0117771347782528"
-        ixy="0.00815174724690121"
-        ixz="6.45200634943833E-05"
-        iyy="0.0106473588161978"
-        iyz="-6.91006905001612E-05"
-        izz="0.0205254157930983" />
-    </inertial>
-    <visual>
-      <origin
-        xyz="0 0 0"
-        rpy="0 0 0" />
-      <geometry>
-        <mesh filename="file:///home/sunshine/project/z_arm_2442c0/install/z_arm_2442c0_model/share/z_arm_2442c0_model/meshes/revolute_1_link.STL"/>
-      </geometry>
-      <material
-        name="">
-        <color
-          rgba="1 1 1 1" />
-      </material>
-    </visual>
-    <collision>
-      <origin
-        xyz="0 0 0"
-        rpy="0 0 0" />
-      <geometry>
-       <mesh filename="file:///home/sunshine/project/z_arm_2442c0/install/z_arm_2442c0_model/share/z_arm_2442c0_model/meshes/revolute_1_link.STL"/>
-      </geometry>
-    </collision>
-  </link>
-  <joint
-    name="lift_revo_joint"
+        xyz="0.0606601004684422 -0.0932567161478479 -0.0341257142535358"
+        rpy="0 0 0" />
+      <mass
+        value="2.3889549988802" />
+      <inertia
+        ixx="0.014531129631885"
+        ixy="0.00746693434928961"
+        ixz="5.15406751826989E-05"
+        iyy="0.00789336402236104"
+        iyz="-7.92546580618748E-05"
+        izz="0.0205254159011504" />
+    </inertial>
+    <visual>
+      <origin
+        xyz="0 0 0"
+        rpy="0 0 0" />
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