Commit message: 修改文件加载路径

File: src/z_arm_2442c0_model/src/urdf/z_arm_2442c0.urdf (robot description, URDF)
Before this commit: robot z_arm_2442c0, 10 links, 9 joints
Links:
- link base_link: geometry collision mesh filename=package://z_arm_2442c0_model/meshes/base_link.STL; visual mesh filename=package://z_arm_2442c0_model/meshes/base_link.STL
- link camera_1_link: geometry collision mesh filename=package://z_arm_2442c0_model/meshes/camera_1_link.STL; visual mesh filename=package://z_arm_2442c0_model/meshes/camera_1_link.STL
- link camera_2_link: geometry collision mesh filename=package://z_arm_2442c0_model/meshes/camera_2_link.STL; visual mesh filename=package://z_arm_2442c0_model/meshes/camera_2_link.STL
- link camera_base_link: geometry collision mesh filename=package://z_arm_2442c0_model/meshes/camera_base_link.STL; visual mesh filename=package://z_arm_2442c0_model/meshes/camera_base_link.STL
- link door_link: geometry collision mesh filename=package://z_arm_2442c0_model/meshes/door_link.STL; visual mesh filename=package://z_arm_2442c0_model/meshes/door_link.STL
- link fixed_link: geometry collision mesh filename=package://z_arm_2442c0_model/meshes/fixed_link.STL; visual mesh filename=package://z_arm_2442c0_model/meshes/fixed_link.STL
- link lift_link: geometry collision mesh filename=package://z_arm_2442c0_model/meshes/lift_link.STL; visual mesh filename=package://z_arm_2442c0_model/meshes/lift_link.STL
- link revolute_1_link: geometry collision mesh filename=package://z_arm_2442c0_model/meshes/revolute_1_link.STL; visual mesh filename=package://z_arm_2442c0_model/meshes/revolute_1_link.STL
- link revolute_2_link: geometry collision mesh filename=package://z_arm_2442c0_model/meshes/revolute_2_link.STL; visual mesh filename=package://z_arm_2442c0_model/meshes/revolute_2_link.STL
- link revolute_3_link: geometry collision mesh filename=package://z_arm_2442c0_model/meshes/revolute_3_link.STL; visual mesh filename=package://z_arm_2442c0_model/meshes/revolute_3_link.STL

File: src/z_arm_2442c0_model/src/urdf/z_arm_2442c0.urdf.xacro (robot description, xacro)
@@ -30,5 +30,5 @@
         rpy="0 0 0" />
       <geometry>
-         <mesh filename="file:///home/sunshine/project/z_arm_2442c0/install/z_arm_2442c0_model/share/z_arm_2442c0_model/meshes/base_link.STL"/>
+         <mesh filename="file://$(find z_arm_2442c0_model)/meshes/base_link.STL"/>
       </geometry>
       <material
@@ -43,5 +43,5 @@
         rpy="0 0 0" />
       <geometry>
-         <mesh filename="file:///home/sunshine/project/z_arm_2442c0/install/z_arm_2442c0_model/share/z_arm_2442c0_model/meshes/base_link.STL"/>
+         <mesh filename="file://$(find z_arm_2442c0_model)/meshes/base_link.STL"/>
       </geometry>
     </collision>
@@ -68,5 +68,5 @@
         rpy="0 0 0" />
       <geometry>
-         <mesh filename="file:///home/sunshine/project/z_arm_2442c0/install/z_arm_2442c0_model/share/z_arm_2442c0_model/meshes/door_link.STL"/>
+         <mesh filename="file://$(find z_arm_2442c0_model)/meshes/door_link.STL"/>
       </geometry>
       <material
@@ -81,5 +81,5 @@
         rpy="0 0 0" />
       <geometry>
-          <mesh filename="file:///home/sunshine/project/z_arm_2442c0/install/z_arm_2442c0_model/share/z_arm_2442c0_model/meshes/door_link.STL"/>
+          <mesh filename="file://$(find z_arm_2442c0_model)/meshes/door_link.STL"/>
       </geometry>
     </collision>
@@ -125,18 +125,18 @@
         rpy="0 0 0" />
       <geometry>
-        <mesh filename="file:///home/sunshine/project/z_arm_2442c0/install/z_arm_2442c0_model/share/z_arm_2442c0_model/meshes/fixed_link.STL"/>
-      </geometry>
-      <material
-        name="">
-        <color
-          rgba="1 1 1 1" />
-      </material>
-    </visual>
-    <collision>
-      <origin
-        xyz="0 0 0"
-        rpy="0 0 0" />
-      <geometry>
-        <mesh filename="file:///home/sunshine/project/z_arm_2442c0/install/z_arm_2442c0_model/share/z_arm_2442c0_model/meshes/fixed_link.STL"/>
+        <mesh filename="file://$(find z_arm_2442c0_model)/meshes/fixed_link.STL"/>
+      </geometry>
+      <material
+        name="">
+        <color
+          rgba="1 1 1 1" />
+      </material>
+    </visual>
+    <collision>
+      <origin
+        xyz="0 0 0"
+        rpy="0 0 0" />
+      <geometry>
+        <mesh filename="file://$(find z_arm_2442c0_model)/meshes/fixed_link.STL"/>
       </geometry>
     </collision>
@@ -176,18 +176,18 @@
         rpy="0 0 0" />
       <geometry>
-        <mesh filename="file:///home/sunshine/project/z_arm_2442c0/install/z_arm_2442c0_model/share/z_arm_2442c0_model/meshes/lift_link.STL"/>
-      </geometry>
-      <material
-        name="">
-        <color
-          rgba="1 1 1 1" />
-      </material>
-    </visual>
-    <collision>
-      <origin
-        xyz="0 0 0"
-        rpy="0 0 0" />
-      <geometry>
-        <mesh filename="file:///home/sunshine/project/z_arm_2442c0/install/z_arm_2442c0_model/share/z_arm_2442c0_model/meshes/lift_link.STL"/>
+        <mesh filename="file://$(find z_arm_2442c0_model)/meshes/lift_link.STL"/>
+      </geometry>
+      <material
+        name="">
+        <color
+          rgba="1 1 1 1" />
+      </material>
+    </visual>
+    <collision>
+      <origin
+        xyz="0 0 0"
+        rpy="0 0 0" />
+      <geometry>
+        <mesh filename="file://$(find z_arm_2442c0_model)/meshes/lift_link.STL"/>
       </geometry>
     </collision>
@@ -229,18 +229,18 @@
         rpy="0 0 0" />
       <geometry>
-        <mesh filename="file:///home/sunshine/project/z_arm_2442c0/install/z_arm_2442c0_model/share/z_arm_2442c0_model/meshes/revolute_1_link.STL"/>
-      </geometry>
-      <material
-        name="">
-        <color
-          rgba="1 1 1 1" />
-      </material>
-    </visual>
-    <collision>
-      <origin
-        xyz="0 0 0"
-        rpy="0 0 0" />
-      <geometry>
-       <mesh filename="file:///home/sunshine/project/z_arm_2442c0/install/z_arm_2442c0_model/share/z_arm_2442c0_model/meshes/revolute_1_link.STL"/>
+        <mesh filename="file://$(find z_arm_2442c0_model)/meshes/revolute_1_link.STL"/>
+      </geometry>
+      <material
+        name="">
+        <color
+          rgba="1 1 1 1" />
+      </material>
+    </visual>
+    <collision>
+      <origin
+        xyz="0 0 0"
+        rpy="0 0 0" />
+      <geometry>
+       <mesh filename="file://$(find z_arm_2442c0_model)/meshes/revolute_1_link.STL"/>
       </geometry>
     </collision>
@@ -282,18 +282,18 @@
         rpy="0 0 0" />
       <geometry>
-        <mesh filename="file:///home/sunshine/project/z_arm_2442c0/install/z_arm_2442c0_model/share/z_arm_2442c0_model/meshes/revolute_2_link.STL"/>
-      </geometry>
-      <material
-        name="">
-        <color
-          rgba="1 1 1 1" />
-      </material>
-    </visual>
-    <collision>
-      <origin
-        xyz="0 0 0"
-        rpy="0 0 0" />
-      <geometry>
-        <mesh filename="file:///home/sunshine/project/z_arm_2442c0/install/z_arm_2442c0_model/share/z_arm_2442c0_model/meshes/revolute_2_link.STL"/>
+        <mesh filename="file://$(find z_arm_2442c0_model)/meshes/revolute_2_link.STL"/>
+      </geometry>
+      <material
+        name="">
+        <color
+          rgba="1 1 1 1" />
+      </material>
+    </visual>
+    <collision>
+      <origin
+        xyz="0 0 0"
+        rpy="0 0 0" />
+      <geometry>
+        <mesh filename="file://$(find z_arm_2442c0_model)/meshes/revolute_2_link.STL"/>
       </geometry>
     </collision>
@@ -335,18 +335,18 @@
         rpy="0 0 0" />
       <geometry>
-        <mesh filename="file:///home/sunshine/project/z_arm_2442c0/install/z_arm_2442c0_model/share/z_arm_2442c0_model/meshes/revolute_3_link.STL"/>
-      </geometry>
-      <material
-        name="">
-        <color
-          rgba="1 1 1 1" />
-      </material>
-    </visual>
-    <collision>
-      <origin
-        xyz="0 0 0"
-        rpy="0 0 0" />
-      <geometry>
-        <mesh filename="file:///home/sunshine/project/z_arm_2442c0/install/z_arm_2442c0_model/share/z_arm_2442c0_model/meshes/revolute_3_link.STL"/>
+        <mesh filename="file://$(find z_arm_2442c0_model)/meshes/revolute_3_link.STL"/>
+      </geometry>
+      <material
+        name="">
+        <color
+          rgba="1 1 1 1" />
+      </material>
+    </visual>
+    <collision>
+      <origin
+        xyz="0 0 0"
+        rpy="0 0 0" />
+      <geometry>
+        <mesh filename="file://$(find z_arm_2442c0_model)/meshes/revolute_3_link.STL"/>
       </geometry>
     </collision>
@@ -388,18 +388,18 @@
         rpy="0 0 0" />
       <geometry>
-        <mesh filename="file:///home/sunshine/project/z_arm_2442c0/install/z_arm_2442c0_model/share/z_arm_2442c0_model/meshes/camera_base_link.STL"/>
-      </geometry>
-      <material
-        name="">
-        <color
-          rgba="1 1 1 1" />
-      </material>
-    </visual>
-    <collision>
-      <origin
-        xyz="0 0 0"
-        rpy="0 0 0" />
-      <geometry>
-        <mesh filename="file:///home/sunshine/project/z_arm_2442c0/install/z_arm_2442c0_model/share/z_arm_2442c0_model/meshes/camera_base_link.STL"/>
+        <mesh filename="file://$(find z_arm_2442c0_model)/meshes/camera_base_link.STL"/>
+      </geometry>
+      <material
+        name="">
+        <color
+          rgba="1 1 1 1" />
+      </material>
+    </visual>
+    <collision>
+      <origin
+        xyz="0 0 0"
+        rpy="0 0 0" />
+      <geometry>
+        <mesh filename="file://$(find z_arm_2442c0_model)/meshes/camera_base_link.STL"/>
       </geometry>
     </collision>
@@ -437,18 +437,18 @@
         rpy="0 0 0" />
       <geometry>
-        <mesh filename="file:///home/sunshine/project/z_arm_2442c0/install/z_arm_2442c0_model/share/z_arm_2442c0_model/meshes/camera_1_link.STL"/>
-      </geometry>
-      <material
-        name="">
-        <color
-          rgba="1 1 1 1" />
-      </material>
-    </visual>
-    <collision>
-      <origin
-        xyz="0 0 0"
-        rpy="0 0 0" />
-      <geometry>
-        <mesh filename="file:///home/sunshine/project/z_arm_2442c0/install/z_arm_2442c0_model/share/z_arm_2442c0_model/meshes/camera_1_link.STL"/>
+        <mesh filename="file://$(find z_arm_2442c0_model)/meshes/camera_1_link.STL"/>
+      </geometry>
+      <material
+        name="">
+        <color
+          rgba="1 1 1 1" />
+      </material>
+    </visual>
+    <collision>
+      <origin
+        xyz="0 0 0"
+        rpy="0 0 0" />
+      <geometry>
+        <mesh filename="file://$(find z_arm_2442c0_model)/meshes/camera_1_link.STL"/>
       </geometry>
     </collision>
@@ -489,18 +489,18 @@
         rpy="0 0 0" />
       <geometry>
-        <mesh filename="file:///home/sunshine/project/z_arm_2442c0/install/z_arm_2442c0_model/share/z_arm_2442c0_model/meshes/camera_2_link.STL"/>
-      </geometry>
-      <material
-        name="">
-        <color
-          rgba="1 1 1 1" />
-      </material>
-    </visual>
-    <collision>
-      <origin
-        xyz="0 0 0"
-        rpy="0 0 0" />
-      <geometry>
-        <mesh filename="file:///home/sunshine/project/z_arm_2442c0/install/z_arm_2442c0_model/share/z_arm_2442c0_model/meshes/camera_2_link.STL"/>
+        <mesh filename="file://$(find z_arm_2442c0_model)/meshes/camera_2_link.STL"/>
+      </geometry>
+      <material
+        name="">
+        <color
+          rgba="1 1 1 1" />
+      </material>
+    </visual>
+    <collision>
+      <origin
+        xyz="0 0 0"
+        rpy="0 0 0" />
+      <geometry>
+        <mesh filename="file://$(find z_arm_2442c0_model)/meshes/camera_2_link.STL"/>
       </geometry>
     </collision>

Commit message: linshi

File: src/z_arm_2442c0_model/src/urdf/z_arm_2442c0.urdf (robot description, URDF)
Before this commit: robot z_arm_2442c0, 12 links, 11 joints
Links:
- removed link camera_1_rot_link
- added link camera_revolute_link, mass 0.118601590695084; collision mesh filename=package://z_arm_2442c0_model/meshes/camera_revolute_link.STL; visual mesh filename=package://z_arm_2442c0_model/meshes/camera_revolute_link.STL
- link camera_base_link: mass 0.321807581331945 -> 0.203205987623318
Joints:
- removed joint camera_1_rot_joint
- added joint camera_revolute_joint: type continuous, parent camera_base_link, child camera_revolute_link, origin xyz=0.141018940058406 7.96433655524172E-05 0.0200000000000001 rpy=0 0 0, axis 0 0 1
- joint camera_1_joint: parent camera_1_rot_link -> camera_revolute_link
- joint camera_2_joint: parent camera_1_rot_link -> camera_revolute_link
- joint camera_3_joint: parent camera_1_rot_link -> camera_revolute_link

Commit message: 修改模型位置参数

File: src/z_arm_2442c0_model/src/urdf/z_arm_2442c0.urdf (robot description, URDF)
Before this commit: robot z_arm_2442c0, 12 links, 11 joints
Joints:
- joint camera_1_joint: origin xyz=0.0234 0.047416 -0.0145 rpy=0 0 0 -> xyz=0.0234 0.047416 0.1 rpy=0 0 0
- joint camera_2_joint: origin xyz=-0.0216 0.047416 -0.0145 rpy=0 0 0 -> xyz=-0.0216 0.047416 0.1 rpy=0 0 0
- joint camera_3_joint: origin xyz=-0.00181 -0.025558 0.029 rpy=0 0 0 -> xyz=-0.00181 -0.025558 0.15 rpy=0 0 0

File: src/z_arm_2442c0_model/src/urdf/z_arm_2442c0.urdf.xacro (robot description, xacro)
@@ -408,16 +408,45 @@
       xyz="0 0 0" />
   </joint>
-  <link name="camera_1_rot_link">
-    <visual>
+  <link name="camera_revolute_link">
+    <inertial>
+      <origin
+        xyz="1.01771558122313E-05 -1.59114604170695E-06 -0.00500000000000023"
+        rpy="0 0 0" />
+      <mass
+        value="0.118601590695084" />
+      <inertia
+        ixx="0.000184097924869798"
+        ixy="2.82010553142919E-06"
+        ixz="-2.91692972568406E-21"
+        iyy="0.000250754763407668"
+        iyz="2.29773777365639E-20"
+        izz="0.000432877616283766" />
+    </inertial>
+    <visual>
+     <origin
+        xyz="0 0 0"
+        rpy="0 0 0" />
+      <geometry>
+        <mesh filename="file://$(find z_arm_2442c0_model)/meshes/camera_revolute_link.STL" />
+      </geometry>
+<material
+        name="">
+        <color
+          rgba="0.792156862745098 0.819607843137255 0.933333333333333 1" />
+      </material>
+    </visual>
+    <collision>
       <origin xyz="0 0 0" rpy="0 0 0"/>
       <geometry>
-        <box size="0.001 0.001 0.001"/> <!-- 可视化一个小点，或直接省略 -->
-      </geometry>
-    </visual>
-  </link>
-  <joint name="camera_1_rot_joint" type="continuous">
-    <origin xyz="0.14534 0 0.13089" rpy="0 0 0"/>
+        <mesh filename="file://$(find z_arm_2442c0_model)/meshes/camera_revolute_link.STL" />
+      </geometry>
+    </collision>
+  </link>
+  <joint name="camera_revolute_joint" type="continuous">
+    <origin
+      xyz="0.141018940058406 7.96433655524172E-05 0.0200000000000001"
+      rpy="0 0 0" />
     <parent link="camera_base_link"/>
-    <child link="camera_1_rot_link"/>
+    <child link="camera_revolute_link"/>
     <axis xyz="0 0 1"/>
   </joint>
@@ -463,7 +492,7 @@
     name="camera_1_joint"
     type="fixed">
-    <origin xyz="0.0234 0.047416 -0.0145" rpy="0 0 0"/>
-    <parent
-      link="camera_1_rot_link" />
+    <origin xyz="0.0234 0.047416 0.1" rpy="0 0 0"/>
+    <parent
+      link="camera_revolute_link" />
     <child
       link="camera_1_link" />
@@ -512,7 +541,7 @@
     name="camera_2_joint"
     type="fixed">
-    <origin xyz="-0.0216 0.047416 -0.0145" rpy="0 0 0"/>
-    <parent
-      link="camera_1_rot_link" />
+    <origin xyz="-0.0216 0.047416 0.1" rpy="0 0 0"/>
+    <parent
+      link="camera_revolute_link" />
     <child
       link="camera_2_link" />
@@ -543,8 +572,8 @@
         <mesh filename="file://$(find z_arm_2442c0_model)/meshes/camera_3_link.STL" />
       </geometry>
-      <material
-        name="">
-        <color
-          rgba="1 1 1 1" />
+<material
+        name="">
+        <color
+          rgba="0.792156862745098 0.819607843137255 0.933333333333333 1" />
       </material>
     </visual>
@@ -561,7 +590,7 @@
     name="camera_3_joint"
     type="fixed">
-  <origin xyz="-0.00181 -0.025558 0.029" rpy="0 0 0"/>
-    <parent
-      link="camera_1_rot_link" />
+  <origin xyz="-0.00181 -0.025558 0.15" rpy="0 0 0"/>
+    <parent
+      link="camera_revolute_link" />
     <child
       link="camera_3_link" />

Commit message: temp

File: src/z_arm_2442c0_model/src/urdf/z_arm_2442c0.urdf (robot description, URDF)
Before this commit: robot z_arm_2442c0, 12 links, 11 joints
Links:
- added link calib_camera_link, mass 0.1; collision box size=0.01 0.01 0.01; visual box size=0.01 0.01 0.01
Joints:
- added joint calib_camera_joint: type fixed, parent camera_base_link, child calib_camera_link, origin xyz=0.237 0 0.01 rpy=0 0 0

File: src/z_arm_2442c0_model/src/urdf/z_arm_2442c0.urdf.xacro (robot description, xacro)
@@ -574,4 +574,29 @@
       xyz="0 0 0" />
   </joint>
+    <!-- 在机械臂末端添加摄像头 -->
+  <link name="calib_camera_link">
+    <visual>
+      <geometry>
+        <box size="0.01 0.01 0.01"/>
+      </geometry>
+      <material name="red">
+        <color rgba="1 0 0 1"/>
+      </material>
+    </visual>
+    <collision>
+      <geometry>
+        <box size="0.01 0.01 0.01"/>
+      </geometry>
+    </collision>
+    <inertial>
+      <mass value="0.1"/>
+      <inertia ixx="0.001" ixy="0.0" ixz="0.0" iyy="0.001" iyz="0.0" izz="0.001"/>
+    </inertial>
+  </link>
+  <joint name="calib_camera_joint" type="fixed">
+    <parent link="camera_base_link"/>  <!-- 替换为您的末端连杆 -->
+    <child link="calib_camera_link"/>
+    <origin xyz="0.2 0 0.1" rpy="0 0 0"/>  <!-- 摄像头位置偏移 -->
+  </joint>
   <gazebo reference="base_link">
         <self_collide>false</self_collide>
@@ -618,4 +643,9 @@
         <self_collide>false</self_collide>
         <gravity>false</gravity>
+    </gazebo>
+    <gazebo reference="calib_camera_link">
+        <self_collide>false</self_collide>
+        <gravity>false</gravity>
+        <material>Gazebo/Red</material>
     </gazebo>
     <gazebo>
@@ -670,25 +700,4 @@
             <state_interface name="velocity"/>
         </joint>
-        <!-- <joint name="camera_1_joint">
-            <command_interface name="position"/>
-            <state_interface name="position">
-                <param name="initial_value">0</param>
-            </state_interface>
-            <state_interface name="velocity"/>
-        </joint>
-        <joint name="camera_2_joint">
-            <command_interface name="position"/>
-            <state_interface name="position">
-                <param name="initial_value">0</param>
-            </state_interface>
-            <state_interface name="velocity"/>
-        </joint>
-        <joint name="camera_3_joint">
-            <command_interface name="position"/>
-            <state_interface name="position">
-                <param name="initial_value">0</param>
-            </state_interface>
-            <state_interface name="velocity"/>
-        </joint> -->
     </ros2_control>
        <!-- 加载ros2_control插件 -->
@@ -700,3 +709,29 @@
         </plugin>
     </gazebo>
+      <!-- Gazebo摄像头插件 -->
+    <gazebo reference="calib_camera_link">
+      <sensor type="camera" name="calib_camera_sensor">
+        <update_rate>30.0</update_rate>
+        <camera name="calib_camera">
+          <horizontal_fov>1.047</horizontal_fov>
+          <image>
+            <width>640</width>
+            <height>480</height>
+            <format>R8G8B8</format>
+          </image>
+          <clip>
+            <near>0.05</near>
+            <far>10.0</far>
+          </clip>
+        </camera>
+        <plugin name="calib_camera_controller" filename="libgazebo_ros_camera.so">
+          <alwaysOn>true</alwaysOn>
+          <updateRate>0.0</updateRate>
+          <cameraName>virtual_camera</cameraName>
+          <imageTopicName>image_raw</imageTopicName>
+          <cameraInfoTopicName>camera_info</cameraInfoTopicName>
+          <frameName>calib_camera_link</frameName>
+        </plugin>
+      </sensor>
+    </gazebo>
 </robot>
